File: Assignment2/Assignment2.kicad_sch (KiCad schematic)
At the start: 33 parts, among them J1 Conn_02x18_Odd_Even, J2 Conn_02x18_Odd_Even, J3 USB_C_Receptacle_USB2.0_14P, J4 Conn_01x02, J5 Screw_Terminal_01x02, U1 RP2040, U2 W25Q128JVS, U3 NCP1117-3.3_SOT223, U4 BMP280, U5 BMI160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

Commit message: Make changes to schematic
Parts:
- removed J1, J2: Conn_02x18_Odd_Even, symbol Connector_Generic:Conn_02x18_Odd_Even
- added D1, D2: D_Schottky, symbol Device:D_Schottky
- added J1: Conn_02x08_Odd_Even, symbol Connector_Generic:Conn_02x08_Odd_Even
Connections:
- net +3V3: now also J1.2 (Pin_2)
- net GND: now also J1.1 (Pin_1), J1.11 (Pin_11), J1.13 (Pin_13), J1.15 (Pin_15), J1.16 (Pin_16), J1.3 (Pin_3), J1.5 (Pin_5), J1.7 (Pin_7), J1.9 (Pin_9)
- net GPIO2: now also J1.4 (Pin_4)
- net GPIO3: now also J1.6 (Pin_6)
- net GPIO4: now also J1.8 (Pin_8)
- net GPIO5: now also J1.10 (Pin_10)
- net SWCLK: now also J1.12 (Pin_12)
- net SWD: now also J1.14 (Pin_14)
- net VBUS: now also D1.1 (K), D2.1 (K); no longer J3.A4 (VBUS), J3.A9 (VBUS), J3.B4 (VBUS), J3.B9 (VBUS), J5.1 (Pin_1)
- net GPIO0: no longer names the net of U1.2 (GPIO0)
- net GPIO1: no longer names the net of U1.3 (GPIO1)
- net GPIO10: no longer names the net of U1.13 (GPIO10)
- net GPIO11: no longer names the net of U1.14 (GPIO11)
- net GPIO12: no longer names the net of U1.15 (GPIO12)
- net GPIO13: no longer names the net of U1.16 (GPIO13)
- net GPIO14: no longer names the net of U1.17 (GPIO14)
- net GPIO15: no longer names the net of U1.18 (GPIO15)
- net GPIO16: no longer names the net of U1.27 (GPIO16)
- net GPIO17: no longer names the net of U1.28 (GPIO17)
- net GPIO18: no longer names the net of U1.29 (GPIO18)
- net GPIO19: no longer names the net of U1.30 (GPIO19)
- net GPIO20: no longer names the net of U1.31 (GPIO20)
- net GPIO21: no longer names the net of U1.32 (GPIO21)
- net GPIO22: no longer names the net of U1.34 (GPIO22)
- net GPIO23: no longer names the net of U1.35 (GPIO23)
- net GPIO24: no longer names the net of U1.36 (GPIO24)
- net GPIO25: no longer names the net of U1.37 (GPIO25)
- net GPIO26_ADC0: no longer names the net of U1.38 (GPIO26_ADC0)
- net GPIO27_ADC1: no longer names the net of U1.39 (GPIO27_ADC1)
- net GPIO28_ADC2: no longer names the net of U1.40 (GPIO28_ADC2)
- net GPIO29_ADC3: no longer names the net of U1.41 (GPIO29_ADC3)
- net GPIO6: no longer names the net of U1.8 (GPIO6)
- net GPIO7: no longer names the net of U1.9 (GPIO7)
- net GPIO8: no longer names the net of U1.11 (GPIO8)
- net GPIO9: no longer names the net of U1.12 (GPIO9)
- net RUN: no longer names the net of U1.26 (RUN)
- new net: D2.2 (A), J3.A4 (VBUS), J3.A9 (VBUS), J3.B4 (VBUS), J3.B9 (VBUS)
- new net: D1.2 (A), J5.1 (Pin_1)
- no-connect marks 8 -> 35

Commit message: Revise Schematic. Set PCB Constraints
Parts:
- removed J1: Conn_02x08_Odd_Even, symbol Connector_Generic:Conn_02x08_Odd_Even
- added J1: Conn_01x03, Connector_PinHeader_2.54mm:PinHeader_1x03_P2.54mm_Vertical, symbol Connector_Generic:Conn_01x03
- added R6, R7, R8: 1k, Resistor_SMD:R_0201_0603Metric, symbol Device:R_Small
- C1, C10, C11, C12, C13, C14, C15, C16, C17, C2, C3, C4, C5, C6, C8, C9: footprint (none) -> Capacitor_SMD:C_0201_0603Metric
- D1, D2: footprint (none) -> Diode_SMD:D_2114_3652Metric
- J3: footprint (none) -> Connector_USB:USB_C_Receptacle_JAE_DX07S016JA1R1500
- J4: footprint (none) -> Connector_PinHeader_2.54mm:PinHeader_1x02_P2.54mm_Vertical
- J5: footprint (none) -> TerminalBlock_Phoenix:TerminalBlock_Phoenix_MPT-0,5-2-2.54_1x02_P2.54mm_Horizontal
- R1, R2, R3, R4, R5: footprint (none) -> Resistor_SMD:R_0201_0603Metric
- Y1: footprint (none) -> Crystal:Crystal_SMD_Abracon_ABM10-4Pin_2.5x2.0mm
Connections:
- net +3V3: now also R6.1, R7.1, R8.1; no longer U4.5 (SDO), U5.1 (SDO), U6.1 (SDO/ADDR)
- net GND: now also J1.3 (Pin_3)
- net SWCLK: now also J1.1 (Pin_1)
- net SWD: now also J1.2 (Pin_2)
- net GPIO4: no longer names the net of U1.6 (GPIO4)
- net GPIO5: no longer names the net of U1.7 (GPIO5)
- new net: R8.2, U6.1 (SDO/ADDR)
- new net: R6.2, U4.5 (SDO)
- new net: R7.2, U5.1 (SDO)
- no-connect marks 35 -> 37
Other:
- note added: "Debug Pins"

Commit message: Arrange PCB elements systematically. Drawing traces still left.
Parts:
- added R9: 1k, Resistor_SMD:R_0201_0603Metric, symbol Device:R_Small
- U6: footprint LGA12_2X2X0P9_ROM -> Audio_Module:LGA12_2X2X0P9_ROM
Connections:
- net +3V3: now also U1.26 (RUN)
- net XOUT: now also R9.2; no longer C13.1, Y1.3
- new net: C13.1, R9.1, Y1.3
- no-connect marks 37 -> 36
Other:
- moved on the sheet: J1, R7, U5

Commit message: Join traces. USB Differential Pair still left.
Parts:
- added C18, C19, C20, C21, C22, C7: 100n, Capacitor_SMD:C_0201_0603Metric, symbol Device:C_Small
Connections:
- net +1V1: now also C18.1
- net +3V3: now also C19.1, C20.1, C21.1, C22.1, C7.1
- net GND: now also C18.2, C19.2, C20.2, C21.2, C22.2, C7.2
